File: A600 68k PLCC to DIP64 v2.kicad_pcb (KiCad board)
At the start: 2 copper layers, 101.9 x 69.2 mm, 9 parts, among them U1 MC68000_PLCC68, U2 68000_SOCKET

Commit message: updated VCC handling
updated PLCC nets to have extra VCC lines from N/C pins to better support thirsty cards like PiStorm.
Parts:
- moved R1 10.8 mm to (113.0, 116.4), turned to 180 degrees
Connections:
- U1 pad 18: Net-(U1-Pad18) -> VCC
- U1 pad 31: Net-(U1-Pad31) -> VCC
Routing:
- net VCC: track 92.0 -> 122.6 mm, vias 1 -> 5
- net GND: track 0.93 -> 11.0 mm, vias 107 -> 93
- net Net-(R1-Pad1): track 11.8 -> 6.58 mm
- added copper zone on B.Cu, net VCC
- added copper zone on F.Cu, net VCC
Other:
- rule pad_to_mask_clearance: 0.05 -> 0
